File: MainBoard/HomeAssistant.kicad_pcb (KiCad board)
At the start: 4 copper layers, 65 x 75 mm, 141 parts, among them J1 10118194-0001LF, J10 Conn_01x02, J11 Conn_01x02, J12 Conn_01x04, J13 Conn_01x04, J14 Conn_01x04, J15 Conn_01x04, J2 XT30PW-M, J3 Conn_01x06, J4 Conn_02x08_Odd_Even, J5 Conn_02x05_Odd_Even, J6 Conn_01x02, J7 Conn_01x02, J8 Conn_01x02, J9 Conn_01x02, Q1 BC848, Q2 BC848, Q3 DMN3023L, Q4 DMN3023L, Q5 DMN3023L, Q6 DMN3023L, Q7 DMN3023L, Q8 DMN3023L, SW1 EVQP2202M, SW2 EVQP2202M, U1 ESP32-S2-MINI-1, U2 CP2102N-A02-GQFN28, U3 LD1117AS33TR, U4 USBLC6-2SC6Y, U5 TPS563201DDCR, U6 TPS563201DDCR, U7 MC74HC365A

Commit message: revision 0.2
Parts:
- removed D1: @CRS06, Diode_SMD:D_SOD-123F
- removed D2: CRS06, Diode_SMD:D_SOD-123F
- added D19: RX, LED_SMD:LED_0805_2012Metric, F.Cu at (67.3, 84.6)
- added D20: TX, LED_SMD:LED_0805_2012Metric, F.Cu at (67.3, 87.4)
- added Q10: SI2347DS, Package_TO_SOT_SMD:TSOT-23, F.Cu at (96.1, 111.2)
- added Q9: SI2347DS, Package_TO_SOT_SMD:TSOT-23, F.Cu at (90.8, 111.2)
- added R51: 470R, Resistor_SMD:R_0805_2012Metric, B.Cu at (67.6, 84.6)
- added R52: 470R, Resistor_SMD:R_0805_2012Metric, B.Cu at (67.6, 87.4)
- added R53: 10K(1%), Resistor_SMD:R_0805_2012Metric, F.Cu at (67.0, 74.3)
- added R54: 10K(1%), Resistor_SMD:R_0805_2012Metric, F.Cu at (73.8, 63.1)
- added R55: 1K, Resistor_SMD:R_0805_2012Metric, F.Cu at (94.9, 114.8)
- added R56: 1K, Resistor_SMD:R_0805_2012Metric, F.Cu at (90.9, 114.8)
- added R57: 100K, Resistor_SMD:R_0805_2012Metric, F.Cu at (96.9, 114.8)
- added R58: 100K, Resistor_SMD:R_0805_2012Metric, F.Cu at (92.9, 114.8)
- C1: value 10uF/25V(20%) -> 0.47uF/35V Tant; footprint Capacitor_SMD:C_0805_2012Metric -> Capacitor_Tantalum_SMD:CP_EIA-3216-18_Kemet-A
- C13, C14: value @0.1uF/50V(10%) -> 0.1uF/50V(10%)
- C4: value 10uF/25V(20%) -> 22uF/6V Tant; footprint Capacitor_SMD:C_0805_2012Metric -> Capacitor_Tantalum_SMD:CP_EIA-3216-18_Kemet-A
- D16: value 3V3_ED RED -> 3V3_ED GREEN
- D17: value 5V_ED RED -> 5V_ED GREEN
- D18: value 5V_ED RED -> 12V_ED GREEN
- D4: value 3V3 RED -> 3V3 BLUE
- R8: value @10K(1%) -> 10K(1%)
- U3: value LD1117AS33TR -> TS2940CW33_RPG; footprint LD1117AS33TR:SOT-223_STM -> TS2940CW33_RPG:VREG_TS2940CW33_RPG
- moved D3 14.9 mm to (104.9, 103.6), turned to 0 degrees
- moved F1 10.5 mm to (98.7, 103.0), turned to 180 degrees
- moved C2 8.88 mm to (91.4, 108.2)
- moved C1 8.75 mm to (91.4, 106.1), turned to 0 degrees
- moved R40 5.90 mm to (114.0, 53.1)
- moved R36 5.86 mm to (115.9, 53.1)
- moved R38 5.81 mm to (117.8, 53.1)
- moved SW2 5.06 mm to (68.6, 69.1), turned to 90 degrees
- moved C4 4.88 mm to (96.4, 106.1), turned to 180 degrees
- moved U3 4.47 mm to (92.6, 99.7), turned to 90 degrees
- moved SW1 4.09 mm to (68.6, 79.7), turned to 90 degrees
- moved D16 2.80 mm to (101.3, 122.8)
- moved D5 1.90 mm to (68.9, 63.2), turned to 180 degrees
- moved C3 1.44 mm to (96.4, 108.2)
- moved D17 1.40 mm to (98.7, 122.8)
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Connections:
- C10 pad 1: /Processor/EN -> /Processor/CHIP_PU
- D5 pad 3: +3V3_FUSED -> Net-(D5-Pad3)
- J2 pad 1: +12V -> GND
- J2 pad 2: GND -> +12V
- R36 pad 1: /IO Connectors/GPIO16 -> /Processor/GPIO16
- R38 pad 1: /IO Connectors/GPIO19 -> /Processor/GPIO19
- R40 pad 1: /IO Connectors/GPIO20 -> /Processor/GPIO20
- R6 pad 2: /Processor/EN -> /Processor/CHIP_PU
- U1 pad 45: /Processor/EN -> /Processor/CHIP_PU
- U3 pad 1: GND -> /Power/VINU3
- U3 pad 2: +3V3 -> GND
- U3 pad 3: /Power/VINU3 -> +3V3
Routing:
- net /Processor/GPIO2: track 106.9 -> 0.00 mm, vias 3 -> 0
- net /IO Connectors/GPIO2: track 0.00 -> 106.9 mm, vias 0 -> 3
- net /Processor/GPIO12: track 0.00 -> 102.1 mm, vias 0 -> 3
- net /IO Connectors/GPIO12: track 102.1 -> 0.00 mm, vias 3 -> 0
- net /Processor/GPIO37/MISO: track 0.00 -> 76.3 mm
- net /IO Connectors/GPIO37/MISO: track 76.3 -> 0.00 mm
- net /Processor/GPIO35/MOSI: track 0.00 -> 76.0 mm
- net /IO Connectors/GPIO35/MOSI: track 76.0 -> 0.00 mm
- net /Processor/GPIO36/CLK: track 0.00 -> 74.0 mm
- net /IO Connectors/GPIO36/CLK: track 74.0 -> 0.00 mm
- net /Processor/U0TXD: track 35.2 -> 76.3 mm, vias 2 -> 4
- net /Processor/GPIO20: track 0.00 -> 35.4 mm, vias 0 -> 2
- net /Processor/U0RXD: track 32.5 -> 66.6 mm, vias 2 -> 4
- net /IO Connectors/GPIO20: track 31.6 -> 0.00 mm, vias 2 -> 0
- net /Processor/CHIP_PU: track 76.5 -> 96.7 mm, vias 3 -> 4
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Other:
- board text added: "ESP32 MQTT Proto Board rev 0.2"
- board text removed: "12V"
- board text removed: "ESP32 MQTT Proto Board rev 0.1"
