File: MainBoard/IO.kicad_sch (KiCad schematic)
At the start: 64 parts, among them J10 Conn_01x02, J11 Conn_01x02, J12 Conn_01x04, J13 Conn_01x04, J14 Conn_01x04, J15 Conn_01x04, J3 Conn_01x06, J4 Conn_02x08_Odd_Even, J5 Conn_02x05_Odd_Even, J6 Conn_01x02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

Commit message: revision 0.2
Parts:
- J4: Name (none) -> DS1023-2*8S21 CONNFLY
- J5: Name (none) -> DS1023-2*5S21 CONNFLY
