File: MainBoard/Power.kicad_sch (KiCad schematic)
At the start: 50 parts, among them J1 10118194-0001LF, J2 XT30PW-M, U3 LD1117AS33TR, U4 USBLC6-2SC6Y, U5 TPS563201DDCR, U6 TPS563201DDCR

Commit message: revision 0.2
Parts:
- removed C1, C4: 10uF/25V(20%), Capacitor_SMD:C_0805_2012Metric, symbol Device:C_Small
- removed D1: @CRS06, Diode_SMD:D_SOD-123F, symbol Device:D_Small
- removed D2: CRS06, Diode_SMD:D_SOD-123F, symbol Device:D_Small
- removed U3: LD1117AS33TR, LD1117AS33TR:SOT-223_STM, symbol 2023-12-15_17-34-47:LD1117AS33TR
- added C1: 0.47uF/35V Tant, Capacitor_Tantalum_SMD:CP_EIA-3216-18_Kemet-A, symbol Device:C_Polarized_Small
- added C4: 22uF/6V Tant, Capacitor_Tantalum_SMD:CP_EIA-3216-18_Kemet-A, symbol Device:C_Polarized_Small
- added Q10, Q9: SI2347DS, Package_TO_SOT_SMD:TSOT-23, symbol Device:Q_PMOS_GSD
- added R55, R56: 1K, Resistor_SMD:R_0805_2012Metric, symbol Device:R_Small
- added R57, R58: 100K, Resistor_SMD:R_0805_2012Metric, symbol Device:R_Small
- added U3: TS2940CW33_RPG, TS2940CW33_RPG:VREG_TS2940CW33_RPG, symbol TS2940CW33_RPG:TS2940CW33_RPG
- D16: value 3V3_ED RED -> 3V3_ED GREEN
- D17: value 5V_ED RED -> 5V_ED GREEN
- D18: value 5V_ED RED -> 12V_ED GREEN
- D4: value 3V3 RED -> 3V3 BLUE
Connections:
- net +12V: now also J2.2 (Pin_2); no longer J2.1 (Pin_1)
- net +12V_FILT: now also Q10.3 (D), R55.1
- net +3V3: now also C4.1, U3.3 (OUT)
- net GND: now also J2.1 (Pin_1), C1.2, C4.2, R57.2, R58.2, U3.2 (GND); no longer J2.2 (Pin_2)
- net VBUS: now also Q9.3 (D), R56.1
- net VINU3: now also C1.1, Q10.2 (S), Q9.2 (S), U3.1 (IN)
- new net R55Q9: Q9.1 (G), R55.2, R58.1
- new net R56Q10: Q10.1 (G), R56.2, R57.1
Other:
- note added: "NOTE! C1 = TAJA474K035R C4 = 293D226X96R3A2TE3"
- moved on the sheet: C2, C25, C26, C3, D17, D3, D4, F1, J2, R48, R5
