File: MainBoard/Processor.kicad_sch (KiCad schematic)
At the start: 27 parts, among them Q1 BC848, Q2 BC848, SW1 EVQP2202M, SW2 EVQP2202M, U1 ESP32-S2-MINI-1, U2 CP2102N-A02-GQFN28

Commit message: revision 0.2
Parts:
- added D19: RX, LED_SMD:LED_0805_2012Metric, symbol Device:LED_Small
- added D20: TX, LED_SMD:LED_0805_2012Metric, symbol Device:LED_Small
- added R51, R52: 470R, Resistor_SMD:R_0805_2012Metric, symbol Device:R_Small
- added R53, R54: 10K(1%), Resistor_SMD:R_0805_2012Metric, symbol Device:R_Small
- C13, C14: value @0.1uF/50V(10%) -> 0.1uF/50V(10%)
- R8: value @10K(1%) -> 10K(1%)
Connections:
- net EN is gone; now on net CHIP_PU: C10.1, R6.2, U1.45 (EN)
- net +3V3_FUSED: now also R53.1, R54.1; no longer D5.3 (VDD)
- net GND: now also D19.1 (K), D20.1 (K)
- net GPIO0: now also R53.2
- net U0RXD: now also R51.1
- net U0TXD: now also R52.1
- new net: D19.2 (A), R51.2
- new net: D5.3 (VDD), R54.2
- new net: D20.2 (A), R52.2
Other:
- moved on the sheet: D5
